Commit message: Add ability to stop at red light

File: catkin_ws/src/auto_rc_car_worlds/urdf/stoplight.xacro.urdf (robot description, URDF)
Before this commit: robot stoplight, 4 links, 3 joints
Links:
- added link green_light_link, mass 1; visual cylinder length=0.001 radius=${sign_radius}
- link base_link: geometry visual cylinder length=${pole_height} radius=0.01
- link light_link: mass 10000 -> 10
- link red_light_link: mass 10000 -> 1; geometry visual cylinder length=0.001 radius=${sign_radius}
Joints:
- added joint green_light_joint: type fixed, parent light_link, child green_light_link, origin xyz=-0.01 0 0 rpy=0 1.5707 0
- joint light_joint: axis (none) -> 0 0 1; limit effort=100 velocity=100 -> lower=-6.3 upper=3.3 effort=100 velocity=100; origin xyz=0 0 1 rpy=0 0 0 -> xyz=0 0 ${pole_height} rpy=0 0 0
- joint red_light_joint: origin xyz=0.01 0 0 rpy=0 0 0 -> xyz=0.01 0 0 rpy=0 1.5707 0
