Commit message: Debugging and dev

File: catkin_ws/src/auto_rc_car_worlds/urdf/pedestrian.urdf.xacro (robot description, xacro)
@@ -42,5 +42,5 @@
     <child link="pedestrian_link"/>
     <axis xyz="1 0 0" />
-    <limit effort="1000" velocity="1000" lower="0" upper="10"/>
+    <limit effort="100000" velocity="1000" lower="0" upper="10"/>
 </joint>
 <transmission name="pedestrian_joint_transmission" type="SimpleTransmission">

Commit message: Development: making some new worlds

File: catkin_ws/src/auto_rc_car_worlds/urdf/pedestrian.urdf.xacro (robot description, xacro)
@@ -156,4 +156,5 @@
   <plugin name="gazebo_ros_control" filename="libgazebo_ros_control.so">
     <robotNamespace>${pedestrian_ns}</robotNamespace>
+    <legacyModeNS>false</legacyModeNS>
   </plugin>
 </gazebo>

File: catkin_ws/src/auto_rc_car_worlds/urdf/stoplight.urdf.xacro (robot description, xacro)
@@ -3,6 +3,8 @@
 <xacro:arg name="light_ns" default="sign0"/>
 <xacro:property name="light_ns" value="$(arg light_ns)"/>
-<xacro:property name="pole_height" value="0.5" />
-<xacro:property name="sign_radius" value="0.2" />
+<xacro:arg name="scale" default="1.0"/>
+<xacro:property name="scale" value="$(arg scale)"/>
+<xacro:property name="pole_height" value="${0.5*scale}" />
+<xacro:property name="sign_radius" value="${0.2*scale}" />
 <link name="world" />
 <joint name="fixed" type="fixed">
@@ -111,4 +113,5 @@
   <plugin name="gazebo_ros_control" filename="libgazebo_ros_control.so">
     <robotNamespace>${light_ns}</robotNamespace>
+    <legacyModeNS>false</legacyModeNS>
   </plugin>
 </gazebo>
