Commit message: Added skid steering. Needs lots of tuning

File: catkin_ws/src/auto_rc_car_description/urdf/car_base.urdf.xacro (robot description, xacro)
@@ -7,5 +7,5 @@
 <xacro:property name="wheel_z_offset" value="-0.1" />
 <xacro:property name="rear_wheel_x_offset" value="-0.2" />
-<xacro:property name="front_wheel_x_offset" value="0.2" />
+<xacro:property name="front_wheel_x_offset" value="0.4" />
 <xacro:property name="pi_2" value="1.5708" />
 <xacro:property name="pi_4" value="0.7854" />
@@ -19,6 +19,6 @@
    <inertial>
      <origin xyz="0 0 0" rpy="0 0 0"/>
-     <mass value="1"/>
-     <inertia ixx="1"  ixy="0"  ixz="0" iyy="10" iyz="0" izz="10" />
+     <mass value="100"/>
+     <inertia ixx="10"  ixy="0"  ixz="0" iyy="10" iyz="0" izz="1" />
    </inertial>
 </xacro:property>
@@ -47,4 +47,13 @@
   </transmission>
 </xacro:macro>
+<xacro:macro name="wheel_params" params="link">
+    <gazebo reference="${link}">
+        <mu1 value="1.0"/>
+        <mu2 value="1.0"/>
+        <kp  value="10000000.0" />
+        <kd  value="2.0" />
+        <material>Gazebo/Black</material>
+    </gazebo>
+</xacro:macro>
 <link name="base_link"/>
 <joint name="base_joint" type="fixed">
@@ -65,6 +74,6 @@
    <inertial>
      <origin xyz="0 0 0" rpy="0 0 0"/>
-     <mass value="10"/>
-     <inertia ixx="100"  ixy="0"  ixz="0" iyy="100" iyz="0" izz="100" />
+     <mass value="100"/>
+     <inertia ixx="100"  ixy="0"  ixz="0" iyy="100" iyz="0" izz="10" />
    </inertial>
    <collision>
@@ -102,8 +111,8 @@
 </link>
 <joint name="right_rear_wheel_joint" type="continuous">
-    <origin xyz="${rear_wheel_x_offset} -${wheel_y_offset} ${wheel_z_offset}" rpy="-${pi_2} 0 0"/>
+    <origin xyz="${rear_wheel_x_offset} -${wheel_y_offset} ${wheel_z_offset}" rpy="${pi_2} 0 0"/>
     <parent link="chassis_link"/>
     <child link="right_rear_wheel_link"/>
-    <axis xyz="0 0 1" />
+    <axis xyz="0 0 -1" />
     <limit effort="10" velocity="100" />
 </joint>
@@ -127,24 +136,9 @@
    </collision>
 </link>
-<joint name="left_front_wheel_turn_joint" type="revolute">
-    <origin xyz="${front_wheel_x_offset} ${wheel_y_offset} ${wheel_z_offset}" rpy="0 0 0"/>
-    <parent link="chassis_link"/>
-    <child link="left_front_wheel_turn_link"/>
-    <axis xyz="0 0 1" />
-    <limit effort="10" velocity="10" lower="-${pi_4}" upper="${pi_4}" />
-</joint>
-<xacro:turn_transmission name="left_front_wheel_turn" />
-<link name="left_front_wheel_turn_link">
-   <inertial>
-     <origin xyz="0 0 0" rpy="0 0 0"/>
-     <mass value="0.1"/>
-     <inertia ixx="0.1"  ixy="0"  ixz="0" iyy="0.1" iyz="0" izz="0.1" />
-   </inertial>
-</link>
 <joint name="left_front_wheel_joint" type="continuous">
-    <origin xyz="0 0 0" rpy="-${pi_2} 0 0"/>
-    <parent link="left_front_wheel_turn_link"/>
+    <origin xyz="${front_wheel_x_offset} ${wheel_y_offset} ${wheel_z_offset}" rpy="${pi_2} 0 0"/>
+    <parent link="chassis_link"/>
     <child link="left_front_wheel_link"/>
-    <axis xyz="0 0 1" />
+    <axis xyz="0 0 -1" />
     <limit effort="10" velocity="100" />
 </joint>
@@ -168,27 +162,11 @@
    </collision>
 </link>
-<joint name="right_front_wheel_turn_joint" type="revolute">
-    <origin xyz="${front_wheel_x_offset} -${wheel_y_offset} ${wheel_z_offset}" rpy="0 0 0"/>
-    <parent link="chassis_link"/>
-    <child link="right_front_wheel_turn_link"/>
-    <axis xyz="0 0 1" />
-    <limit effort="10" velocity="10" lower="-${pi_4}" upper="${pi_4}" />
-</joint>
-<xacro:turn_transmission name="right_front_wheel_turn" />
-<link name="right_front_wheel_turn_link">
-   <inertial>
-     <origin xyz="0 0 0" rpy="0 0 0"/>
-     <mass value="0.1"/>
-     <inertia ixx="0.1"  ixy="0"  ixz="0" iyy="0.1" iyz="0" izz="0.1" />
-   </inertial>
-</link>
 <joint name="right_front_wheel_joint" type="continuous">
-    <origin xyz="0 0 0" rpy="-${pi_2} 0 0"/>
-    <parent link="right_front_wheel_turn_link"/>
+    <origin xyz="${front_wheel_x_offset} -${wheel_y_offset} ${wheel_z_offset}" rpy="${pi_2} 0 0"/>
+    <parent link="chassis_link"/>
     <child link="right_front_wheel_link"/>
-    <axis xyz="0 0 1" />
-    <limit effort="10" velocity="100" />
-</joint>
-<xacro:wheel_transmission name="right_front_wheel" />
+    <axis xyz="0 0 -1" />
+    <limit effort="10" velocity="100" />
+</joint>
 <link name="right_front_wheel_link">
     <visual>
@@ -214,43 +192,8 @@
   </plugin>
 </gazebo>
-<gazebo reference="chassis_link">
-  <mu1 value="0.0"/>
-  <mu2 value="0.0"/>
-  <kp  value="10000000.0" />
-  <kd  value="1.0" />
-  <material>Gazebo/Blue</material>
-</gazebo>
-<gazebo reference="left_rear_wheel_link">
-  <mu1 value="100.0"/>
-  <mu2 value="50.0"/>
-  <kp  value="10000000.0" />
-  <kd  value="1.0" />
-  <fdir1 value="1 0 0"/>
-  <material>Gazebo/Black</material>
-</gazebo>
-<gazebo reference="right_rear_wheel_link">
-  <mu1 value="100.0"/>
-  <mu2 value="50.0"/>
-  <kp  value="10000000.0" />
-  <kd  value="1.0" />
-  <fdir1 value="1 0 0"/>
-  <material>Gazebo/Black</material>
-</gazebo>
-<gazebo reference="left_front_wheel_link">
-  <mu1 value="100.0"/>
-  <mu2 value="50.0"/>
-  <kp  value="10000000.0" />
-  <kd  value="1.0" />
-  <fdir1 value="0 0 1"/>
-  <material>Gazebo/Black</material>
-</gazebo>
-<gazebo reference="right_front_wheel_link">
-  <mu1 value="100.0"/>
-  <mu2 value="50.0"/>
-  <kp  value="10000000.0" />
-  <kd  value="1.0" />
-  <fdir1 value="0 0 1"/>
-  <material>Gazebo/Black</material>
-</gazebo>
+<xacro:wheel_params link="left_rear_wheel_link"/>
+<xacro:wheel_params link="right_rear_wheel_link"/>
+<xacro:wheel_params link="left_front_wheel_link"/>
+<xacro:wheel_params link="right_front_wheel_link"/>
 <gazebo>
   <plugin name="skid_steer_drive_controller" filename="libgazebo_ros_skid_steer_drive.so">
@@ -264,5 +207,5 @@
     <wheelDiameter>0.215</wheelDiameter>
     <robotBaseFrame>chassis_link</robotBaseFrame>
-    <torque>20</torque>
+    <torque>1000</torque>
     <topicName>cmd_vel</topicName>
     <broadcastTF>false</broadcastTF>

Commit message: Starting to set up sensors

File: catkin_ws/src/auto_rc_car_description/urdf/car_base.urdf.xacro (robot description, xacro)
@@ -16,11 +16,27 @@
   <cylinder length="0.05" radius="0.1" />
 </xacro:property>
+<xacro:property name="chassis_inertia">
+   <inertial>
+     <origin xyz="0 0 0" rpy="0 0 0"/>
+     <mass value="100"/>
+     <inertia ixx="100"  ixy="0"  ixz="0" iyy="100" iyz="0" izz="10" />
+   </inertial>
+</xacro:property>
 <xacro:property name="wheel_inertia">
    <inertial>
      <origin xyz="0 0 0" rpy="0 0 0"/>
-     <mass value="100"/>
+     <mass value="1"/>
      <inertia ixx="10"  ixy="0"  ixz="0" iyy="10" iyz="0" izz="1" />
    </inertial>
 </xacro:property>
+<xacro:macro name="wheel_params" params="link">
+    <gazebo reference="${link}">
+        <mu1 value="1.0"/>
+        <mu2 value="1.0"/>
+        <kp  value="10000000.0" />
+        <kd  value="2.0" />
+        <material>Gazebo/Black</material>
+    </gazebo>
+</xacro:macro>
 <xacro:macro name="wheel_transmission" params="name">
   <transmission name="${name}_transmission" type="SimpleTransmission">
@@ -47,13 +63,4 @@
   </transmission>
 </xacro:macro>
-<xacro:macro name="wheel_params" params="link">
-    <gazebo reference="${link}">
-        <mu1 value="1.0"/>
-        <mu2 value="1.0"/>
-        <kp  value="10000000.0" />
-        <kd  value="2.0" />
-        <material>Gazebo/Black</material>
-    </gazebo>
-</xacro:macro>
 <link name="base_link"/>
 <joint name="base_joint" type="fixed">
@@ -72,9 +79,5 @@
         </material>
    </visual>
-   <inertial>
-     <origin xyz="0 0 0" rpy="0 0 0"/>
-     <mass value="100"/>
-     <inertia ixx="100"  ixy="0"  ixz="0" iyy="100" iyz="0" izz="10" />
-   </inertial>
+    <xacro:insert_block name="chassis_inertia" />
    <collision>
      <origin xyz="0 0 0" rpy="0 0 0"/>
@@ -162,4 +165,5 @@
    </collision>
 </link>
+<xacro:wheel_transmission name="right_front_wheel" />
 <joint name="right_front_wheel_joint" type="continuous">
     <origin xyz="${front_wheel_x_offset} -${wheel_y_offset} ${wheel_z_offset}" rpy="${pi_2} 0 0"/>
@@ -212,3 +216,88 @@
   </plugin>
 </gazebo>
+<joint name="hoyuko_fixed_joint" type="fixed">
+    <origin xyz="0 0 0.25" rpy="0 0 0"/>
+    <parent link="chassis_link"/>
+    <child link="hoyuko_laser_link"/>
+    <axis xyz="0 0 1" />
+</joint>
+<link name="hoyuko_laser_link">
+   <inertial>
+     <origin xyz="0 0 0" rpy="0 0 0"/>
+     <mass value="1"/>
+     <inertia ixx="10"  ixy="0"  ixz="0" iyy="10" iyz="0" izz="1" />
+   </inertial>
+</link>
+<xacro:unless value="$(optenv DISABLE_GAZEBO_LASER false)">
+  <gazebo reference="hoyuko_laser_link">
+    <material>Gazebo/Grey</material>
+    <sensor type="ray" name="hokuyo_sensor">
+      <pose>0 0 0.0124 0 0 0</pose>
+      <visualize>false</visualize>
+      <update_rate>40</update_rate>
+      <ray>
+        <scan>
+          <horizontal>
+            <samples>1081</samples>
+            <resolution>1</resolution>
+            <min_angle>-2.3561944902</min_angle>
+            <max_angle>2.3561944902</max_angle>
+          </horizontal>
+        </scan>
+        <range>
+          <min>0.1</min>
+          <max>10.0</max>
+          <resolution>0.01</resolution>
+        </range>
+        <noise>
+          <mean>0.0</mean>
+          <stddev>0.01</stddev>
+        </noise>
+      </ray>
+      <plugin name="gazebo_ros_hokuyo_controller" filename="libgazebo_ros_laser.so">
+        <topicName>racecar/out/laser_scan</topicName>
+        <frameName>hoyuko_laser_link</frameName>
+      </plugin>
+    </sensor>
+  </gazebo>
+</xacro:unless>
+<xacro:unless value="$(optenv DISABLE_GAZEBO_CAMERA false)">
+  <gazebo reference="hoyuko_laser_link">
+    <sensor type="camera" name="camera">
+      <update_rate>30.0</update_rate>
+      <!-- math.atan(320 / 687.8065795898438) * 2 -->
+      <camera name="camera">
+        <horizontal_fov>0.8709216071359963</horizontal_fov>
+        <image>
+          <width>640</width>
+          <height>480</height>
+          <format>B8G8R8</format>
+        </image>
+        <clip>
+          <near>0.02</near>
+          <far>300</far>
+        </clip>
+        <noise>
+          <type>gaussian</type>
+          <mean>0.0</mean>
+          <stddev>0.007</stddev>
+        </noise>
+      </camera>
+      <plugin name="camera_controller" filename="libgazebo_ros_camera.so">
+        <alwaysOn>true</alwaysOn>
+        <updateRate>30.0</updateRate>
+        <cameraName>/camera/zed</cameraName>
+        <imageTopicName>rgb/image_rect_color</imageTopicName>
+        <cameraInfoTopicName>rgb/camera_info</cameraInfoTopicName>
+        <frameName>hoyuko_laser_link</frameName>
+        <hackBaseline>0</hackBaseline><!-- set this to 0.12 for the second camera -->
+        <distortionK1>0.0</distortionK1>
+        <distortionK2>0.0</distortionK2>
+        <distortionK3>0.0</distortionK3>
+        <distortionT1>0.0</distortionT1>
+        <distortionT2>0.0</distortionT2>
+      </plugin>
+    </sensor>
+  </gazebo>
+</xacro:unless>
 </robot>

Commit message: Fixed sim camera and created camera launch file

File: catkin_ws/src/auto_rc_car_description/urdf/car_base.urdf.xacro (robot description, xacro)
@@ -229,4 +229,17 @@
    </inertial>
 </link>
+<joint name="kinect_fixed_joint" type="fixed">
+    <origin xyz="0 0 0.25" rpy="0 0 0"/>
+    <parent link="chassis_link"/>
+    <child link="kinect_link"/>
+    <axis xyz="0 0 1" />
+</joint>
+<link name="kinect_link">
+   <inertial>
+     <origin xyz="0 0 0" rpy="0 0 0"/>
+     <mass value="1"/>
+     <inertia ixx="10"  ixy="0"  ixz="0" iyy="10" iyz="0" izz="1" />
+   </inertial>
+</link>
 <xacro:unless value="$(optenv DISABLE_GAZEBO_LASER false)">
   <gazebo reference="hoyuko_laser_link">
@@ -262,42 +275,55 @@
   </gazebo>
 </xacro:unless>
-<xacro:unless value="$(optenv DISABLE_GAZEBO_CAMERA false)">
-  <gazebo reference="hoyuko_laser_link">
-    <sensor type="camera" name="camera">
-      <update_rate>30.0</update_rate>
-      <!-- math.atan(320 / 687.8065795898438) * 2 -->
-      <camera name="camera">
-        <horizontal_fov>0.8709216071359963</horizontal_fov>
-        <image>
-          <width>640</width>
-          <height>480</height>
-          <format>B8G8R8</format>
-        </image>
-        <clip>
-          <near>0.02</near>
-          <far>300</far>
-        </clip>
-        <noise>
-          <type>gaussian</type>
-          <mean>0.0</mean>
-          <stddev>0.007</stddev>
-        </noise>
-      </camera>
-      <plugin name="camera_controller" filename="libgazebo_ros_camera.so">
-        <alwaysOn>true</alwaysOn>
-        <updateRate>30.0</updateRate>
-        <cameraName>/camera/zed</cameraName>
-        <imageTopicName>rgb/image_rect_color</imageTopicName>
-        <cameraInfoTopicName>rgb/camera_info</cameraInfoTopicName>
-        <frameName>hoyuko_laser_link</frameName>
-        <hackBaseline>0</hackBaseline><!-- set this to 0.12 for the second camera -->
-        <distortionK1>0.0</distortionK1>
-        <distortionK2>0.0</distortionK2>
-        <distortionK3>0.0</distortionK3>
-        <distortionT1>0.0</distortionT1>
-        <distortionT2>0.0</distortionT2>
-      </plugin>
+  <joint name="camera_optical_joint" type="fixed">
+    <!-- these values have to be these values otherwise the gazebo camera
+        image won't be aligned properly with the frame it is supposedly
+        originating from -->
+    <origin xyz="0 0 0" rpy="${-pi/2} 0 ${-pi/2}"/>
+    <parent link="kinect_link"/>
+    <child link="camera_link_optical"/>
+  </joint>
+  <link name="camera_link_optical">
+  </link>
+  <gazebo reference="kinect_link">
+        <sensor name="camera" type="depth">
+        <pose>0 0 0 0 0 0</pose>
+        <visualize>true</visualize>
+        <update_rate>20</update_rate>
+        <camera>
+          <horizontal_fov>1.047198</horizontal_fov>
+          <image>
+            <width>640</width>
+            <height>480</height>
+            <format>R8G8B8</format>
+          </image>
+          <clip>
+            <near>0.05</near>
+            <far>3</far>
+          </clip>
+        </camera>
+    <plugin name="camera_plugin" filename="libgazebo_ros_openni_kinect.so">
+      <baseline>0.2</baseline>
+      <alwaysOn>true</alwaysOn>
+      <updateRate>30.0</updateRate>
+      <cameraName>sim_depth_camera</cameraName>
+      <imageTopicName>/racecar/out/stereo_camera/rgb/image</imageTopicName>
+      <cameraInfoTopicName>/racecar/out/stereo_camera/rgb/camera_info</cameraInfoTopicName>
+      <depthImageTopicName>/racecar/out/stereo_camera/depth/image</depthImageTopicName>
+      <depthImageInfoTopicName>/racecar/out/stereo_camera/depth/camera_info</depthImageInfoTopicName>
+      <pointCloudTopicName>/racecar/out/stereo_camera/depth_cloud/points</pointCloudTopicName>
+      <frameName>camera_link_optical</frameName>
+      <pointCloudCutoff>0.05</pointCloudCutoff>
+      <distortionK1>0</distortionK1>
+      <distortionK2>0</distortionK2>
+      <distortionK3>0</distortionK3>
+      <distortionT1>0</distortionT1>
+      <distortionT2>0</distortionT2>
+      <CxPrime>0</CxPrime>
+      <Cx>0</Cx>
+      <Cy>0</Cy>
+      <focalLength>0</focalLength>
+      <hackBaseline>0</hackBaseline>
+    </plugin>
     </sensor>
-  </gazebo>
-</xacro:unless>
+    </gazebo>
 </robot>

Commit message: misc changes

File: catkin_ws/src/auto_rc_car_description/urdf/car_base.urdf.xacro (robot description, xacro)
@@ -293,6 +293,6 @@
           <horizontal_fov>1.047198</horizontal_fov>
           <image>
-            <width>640</width>
-            <height>480</height>
+            <width>320</width>
+            <height>240</height>
             <format>R8G8B8</format>
           </image>

File: catkin_ws/src/auto_rc_car_worlds/urdf/circle_track.urdf (robot description, URDF)
Before this commit: robot circle_track, 2 links, 1 joints
Joints:
- removed joint world_joint
- added joint fixed: type fixed, parent world, child circle_base_link

Commit message: Changed up visualization

File: catkin_ws/src/auto_rc_car_description/urdf/car_base.urdf.xacro (robot description, xacro)
@@ -32,8 +32,8 @@
 <xacro:macro name="wheel_params" params="link">
     <gazebo reference="${link}">
-        <mu1 value="1.0"/>
-        <mu2 value="1.0"/>
+        <mu1 value="10.0"/>
+        <mu2 value="10.0"/>
         <kp  value="10000000.0" />
-        <kd  value="2.0" />
+        <kd  value="5.0" />
         <material>Gazebo/Black</material>
     </gazebo>
@@ -43,8 +43,8 @@
     <type>transmission_interface/SimpleTransmission</type>
     <joint name="${name}_joint">
-      <hardwareInterface>EffortJointInterface</hardwareInterface>
+      <hardwareInterface>hardware_interface/EffortJointInterface</hardwareInterface>
     </joint>
     <actuator name="${name}_motor">
-      <hardwareInterface>EffortJointInterface</hardwareInterface>
+      <hardwareInterface>hardware_interface/EffortJointInterface</hardwareInterface>
       <mechanicalReduction>1</mechanicalReduction>
     </actuator>
@@ -87,12 +87,45 @@
    </collision>
 </link>
-<joint name="left_rear_wheel_joint" type="continuous">
-    <origin xyz="${rear_wheel_x_offset} ${wheel_y_offset} ${wheel_z_offset}" rpy="${pi_2} 0 0"/>
+<joint name="rear_speed_joint" type="continuous">
+  <origin xyz="${rear_wheel_x_offset} 0 ${wheel_z_offset}" rpy="0 0 0"/>
     <parent link="chassis_link"/>
+    <child link="rear_speed_link"/>
+    <axis xyz="0 1 0" />
+    <limit effort="100" velocity="100" />
+</joint>
+<transmission name="speed_joint_transmission" type="SimpleTransmission">
+  <type>transmission_interface/SimpleTransmission</type>
+  <joint name="rear_speed_joint">
+    <hardwareInterface>EffortJointInterface</hardwareInterface>
+  </joint>
+  <actuator name="rear_speed_joint_motor">
+    <hardwareInterface>EffortJointInterface</hardwareInterface>
+    <mechanicalReduction>1</mechanicalReduction>
+  </actuator>
+</transmission>
+<link name="rear_speed_link">
+   <inertial>
+     <origin xyz="0 0 0" rpy="0 0 0"/>
+     <mass value="1"/>
+     <inertia ixx="10"  ixy="0"  ixz="0" iyy="1" iyz="0" izz="10" />
+   </inertial>
+    <visual>
+        <origin xyz="0 0 0" rpy="${pi/2.0} 0 0" />
+        <geometry>
+            <cylinder radius="0.01" length="0.5"/>
+        </geometry>
+            <material name="Cyan">
+            <color rgba="0 1.0 1.0 1.0"/>
+        </material>
+   </visual>
+</link>
+<joint name="left_rear_wheel_joint" type="fixed">
+    <origin xyz="0 ${wheel_y_offset} 0" rpy="${pi/2.0} 0 0"/>
+    <parent link="rear_speed_link"/>
     <child link="left_rear_wheel_link"/>
     <axis xyz="0 0 -1" />
     <limit effort="10" velocity="100" />
 </joint>
-<xacro:wheel_transmission name="left_rear_wheel" />
+<!--<xacro:wheel_transmission name="left_rear_wheel" />-->
 <link name="left_rear_wheel_link">
     <visual>
@@ -113,12 +146,12 @@
    </collision>
 </link>
-<joint name="right_rear_wheel_joint" type="continuous">
-    <origin xyz="${rear_wheel_x_offset} -${wheel_y_offset} ${wheel_z_offset}" rpy="${pi_2} 0 0"/>
-    <parent link="chassis_link"/>
+<joint name="right_rear_wheel_joint" type="fixed">
+    <origin xyz="0 -${wheel_y_offset} 0" rpy="${pi/2.0} 0 0"/>
+    <parent link="rear_speed_link"/>
     <child link="right_rear_wheel_link"/>
     <axis xyz="0 0 -1" />
     <limit effort="10" velocity="100" />
 </joint>
-<xacro:wheel_transmission name="right_rear_wheel" />
+<!--<xacro:wheel_transmission name="right_rear_wheel" />-->
 <link name="right_rear_wheel_link">
     <visual>
@@ -139,7 +172,40 @@
    </collision>
 </link>
+<joint name="front_steer_joint" type="revolute">
+  <origin xyz="${front_wheel_x_offset} 0 ${wheel_z_offset}" rpy="0 0 0"/>
+    <parent link="chassis_link"/>
+    <child link="front_steer_link"/>
+    <axis xyz="0 0 1" />
+    <limit upper="0.5" lower="-0.5" effort="100" velocity="10" />
+</joint>
+<transmission name="steer_joint_transmission" type="SimpleTransmission">
+  <type>transmission_interface/SimpleTransmission</type>
+  <joint name="front_steer_joint">
+    <hardwareInterface>EffortJointInterface</hardwareInterface>
+  </joint>
+  <actuator name="front_steer_joint_motor">
+    <hardwareInterface>EffortJointInterface</hardwareInterface>
+    <mechanicalReduction>1</mechanicalReduction>
+  </actuator>
+</transmission>
+<link name="front_steer_link">
+   <inertial>
+     <origin xyz="0 0 0" rpy="0 0 0"/>
+     <mass value="1"/>
+     <inertia ixx="10"  ixy="0"  ixz="0" iyy="10" iyz="0" izz="1" />
+   </inertial>
+    <visual>
+        <origin xyz="0 0 0" rpy="0 0 0" />
+        <geometry>
+            <box size="0.05 0.4 0.05" />
+        </geometry>
+            <material name="Cyan">
+            <color rgba="0 1.0 1.0 1.0"/>
+        </material>
+   </visual>
+</link>
 <joint name="left_front_wheel_joint" type="continuous">
-    <origin xyz="${front_wheel_x_offset} ${wheel_y_offset} ${wheel_z_offset}" rpy="${pi_2} 0 0"/>
-    <parent link="chassis_link"/>
+    <origin xyz="0 ${wheel_y_offset} 0" rpy="${pi_2} 0 0"/>
+    <parent link="front_steer_link"/>
     <child link="left_front_wheel_link"/>
     <axis xyz="0 0 -1" />
@@ -167,6 +233,6 @@
 <xacro:wheel_transmission name="right_front_wheel" />
 <joint name="right_front_wheel_joint" type="continuous">
-    <origin xyz="${front_wheel_x_offset} -${wheel_y_offset} ${wheel_z_offset}" rpy="${pi_2} 0 0"/>
-    <parent link="chassis_link"/>
+    <origin xyz="0 -${wheel_y_offset} 0" rpy="${pi_2} 0 0"/>
+    <parent link="front_steer_link"/>
     <child link="right_front_wheel_link"/>
     <axis xyz="0 0 -1" />
@@ -195,4 +261,14 @@
     <robotNamespace>/racecar/internal</robotNamespace>
   </plugin>
+  <plugin name="p3d_base_controller" filename="libgazebo_ros_p3d.so">
+      <alwaysOn>true</alwaysOn>
+      <updateRate>50.0</updateRate>
+      <bodyName>base_link</bodyName>
+      <topicName>/racecar/internal/sim_only/global_pos</topicName>
+      <gaussianNoise>0.01</gaussianNoise>
+      <frameName>world</frameName>
+      <xyzOffsets>0 0 0</xyzOffsets>
+      <rpyOffsets>0 0 0</rpyOffsets>
+    </plugin>
 </gazebo>
 <xacro:wheel_params link="left_rear_wheel_link"/>
@@ -200,20 +276,4 @@
 <xacro:wheel_params link="left_front_wheel_link"/>
 <xacro:wheel_params link="right_front_wheel_link"/>
-<gazebo>
-  <plugin name="skid_steer_drive_controller" filename="libgazebo_ros_skid_steer_drive.so">
-    <updateRate>100.0</updateRate>
-    <robotNamespace>/racecar/in</robotNamespace>
-    <leftFrontJoint>left_front_wheel_joint</leftFrontJoint>
-    <rightFrontJoint>right_front_wheel_joint</rightFrontJoint>
-    <leftRearJoint>left_rear_wheel_joint</leftRearJoint>
-    <rightRearJoint>right_rear_wheel_joint</rightRearJoint>
-    <wheelSeparation>0.4</wheelSeparation>
-    <wheelDiameter>0.215</wheelDiameter>
-    <robotBaseFrame>chassis_link</robotBaseFrame>
-    <torque>1000</torque>
-    <topicName>cmd_vel</topicName>
-    <broadcastTF>false</broadcastTF>
-  </plugin>
-</gazebo>
 <joint name="hoyuko_fixed_joint" type="fixed">
     <origin xyz="0 0 0.25" rpy="0 0 0"/>
