Commit message: Size car

File: catkin_ws/src/auto_rc_car_description/urdf/car_base.urdf.xacro (robot description, xacro)
@@ -4,15 +4,13 @@
 mit-racecar/racecar_gazebo
 -->
-<xacro:property name="wheel_y_offset" value="0.2" />
-<xacro:property name="wheel_z_offset" value="-0.1" />
-<xacro:property name="rear_wheel_x_offset" value="-0.2" />
-<xacro:property name="front_wheel_x_offset" value="0.4" />
+<!-- Set Origin: Center of body lengthwise, height of ~middle of the gearbox -->
+<xacro:property name="wheel_y_offset" value="0.115" />
+<xacro:property name="wheel_z_offset" value="-0.03" />
+<xacro:property name="rear_wheel_x_offset" value="-0.14" />
+<xacro:property name="front_wheel_x_offset" value="0.14" />
 <xacro:property name="pi_2" value="1.5708" />
 <xacro:property name="pi_4" value="0.7854" />
 <xacro:property name="chassis_geometry">
-  <box size="0.5 0.3 0.2" />
-</xacro:property>
-<xacro:property name="wheel_geometry">
-  <cylinder length="0.05" radius="0.1" />
+  <box size="0.4 0.13 0.05" />
 </xacro:property>
 <xacro:property name="chassis_inertia">
@@ -23,43 +21,54 @@
    </inertial>
 </xacro:property>
-<xacro:property name="wheel_inertia">
-   <inertial>
-     <origin xyz="0 0 0" rpy="0 0 0"/>
-     <mass value="1"/>
-     <inertia ixx="10"  ixy="0"  ixz="0" iyy="10" iyz="0" izz="1" />
-   </inertial>
-</xacro:property>
-<xacro:macro name="wheel_params" params="link">
-    <gazebo reference="${link}">
-        <mu1 value="10.0"/>
-        <mu2 value="10.0"/>
-        <kp  value="10000000.0" />
-        <kd  value="5.0" />
-        <material>Gazebo/Black</material>
-    </gazebo>
+<xacro:macro name="wheel" params="name y_offset parent j_type">
+  <joint name="${name}_joint" type="${j_type}">
+    <origin xyz="0 ${y_offset} 0" rpy="${pi_2} 0 0"/>
+    <parent link="${parent}"/>
+    <child link="${name}_link"/>
+    <axis xyz="0 0 -1" />
+    <limit effort="10" velocity="100" />
+  </joint>
+  <link name="${name}_link">
+    <visual>
+      <origin xyz="0 0 0" rpy="0 0 0" />
+      <geometry>
+        <cylinder length="0.05" radius="0.055" />
+      </geometry>
+      <material name="Black">
+        <color rgba="0 0 0 1"/>
+      </material>
+    </visual>
+    <inertial>
+      <origin xyz="0 0 0" rpy="0 0 0"/>
+      <mass value="1"/>
+      <inertia ixx="10"  ixy="0"  ixz="0" iyy="10" iyz="0" izz="1" />
+    </inertial>
+    <collision>
+      <origin xyz="0 0 0" rpy="0 0 0"/>
+      <geometry>
+        <cylinder length="0.05" radius="0.1" />
+      </geometry>
+    </collision>
+  </link>
+    <gazebo reference="${name}_link">
+      <mu1 value="10.0"/>
+      <mu2 value="10.0"/>
+      <kp  value="10000000.0" />
+      <kd  value="5.0" />
+      <material>Gazebo/Black</material>
+  </gazebo>
 </xacro:macro>
-<xacro:macro name="wheel_transmission" params="name">
-  <transmission name="${name}_transmission" type="SimpleTransmission">
-    <type>transmission_interface/SimpleTransmission</type>
-    <joint name="${name}_joint">
-      <hardwareInterface>hardware_interface/EffortJointInterface</hardwareInterface>
-    </joint>
-    <actuator name="${name}_motor">
-      <hardwareInterface>hardware_interface/EffortJointInterface</hardwareInterface>
-      <mechanicalReduction>1</mechanicalReduction>
-    </actuator>
-  </transmission>
-</xacro:macro>
-<xacro:macro name="turn_transmission" params="name">
-  <transmission name="${name}_transmission" type="SimpleTransmission">
-    <type>transmission_interface/SimpleTransmission</type>
-    <joint name="${name}_joint">
-      <hardwareInterface>EffortJointInterface</hardwareInterface>
-    </joint>
-    <actuator name="${name}_motor">
-      <hardwareInterface>EffortJointInterface</hardwareInterface>
-      <mechanicalReduction>1</mechanicalReduction>
-    </actuator>
-  </transmission>
+<xacro:macro name="slipping_wheel" params="name y_offset parent j_type">
+  <xacro:wheel name="${name}" y_offset="${y_offset}" parent="${parent}" j_type="${j_type}"/>
+  <transmission name="${name}_joint_transmission" type="SimpleTransmission">
+  <type>transmission_interface/SimpleTransmission</type>
+  <joint name="${name}_joint">
+    <hardwareInterface>EffortJointInterface</hardwareInterface>
+  </joint>
+  <actuator name="${name}_joint_motor">
+    <hardwareInterface>EffortJointInterface</hardwareInterface>
+    <mechanicalReduction>1</mechanicalReduction>
+  </actuator>
+</transmission>
 </xacro:macro>
 <link name="base_link"/>
@@ -113,5 +122,5 @@
         <origin xyz="0 0 0" rpy="${pi/2.0} 0 0" />
         <geometry>
-            <cylinder radius="0.01" length="0.5"/>
+            <cylinder radius="0.01" length="0.18"/>
         </geometry>
             <material name="Cyan">
@@ -120,56 +129,6 @@
    </visual>
 </link>
-<joint name="left_rear_wheel_joint" type="fixed">
-    <origin xyz="0 ${wheel_y_offset} 0" rpy="${pi/2.0} 0 0"/>
-    <parent link="rear_speed_link"/>
-    <child link="left_rear_wheel_link"/>
-    <axis xyz="0 0 -1" />
-    <limit effort="10" velocity="100" />
-</joint>
-<!--<xacro:wheel_transmission name="left_rear_wheel" />-->
-<link name="left_rear_wheel_link">
-    <visual>
-        <origin xyz="0 0 0" rpy="0 0 0" />
-        <geometry>
-            <xacro:insert_block name="wheel_geometry" />
-        </geometry>
-            <material name="Black">
-            <color rgba="0 0 0 1"/>
-        </material>
-   </visual>
-   <xacro:insert_block name="wheel_inertia" />
-   <collision>
-     <origin xyz="0 0 0" rpy="0 0 0"/>
-     <geometry>
-       <xacro:insert_block name="wheel_geometry" />
-     </geometry>
-   </collision>
-</link>
-<joint name="right_rear_wheel_joint" type="fixed">
-    <origin xyz="0 -${wheel_y_offset} 0" rpy="${pi/2.0} 0 0"/>
-    <parent link="rear_speed_link"/>
-    <child link="right_rear_wheel_link"/>
-    <axis xyz="0 0 -1" />
-    <limit effort="10" velocity="100" />
-</joint>
-<!--<xacro:wheel_transmission name="right_rear_wheel" />-->
-<link name="right_rear_wheel_link">
-    <visual>
-        <origin xyz="0 0 0" rpy="0 0 0" />
-        <geometry>
-            <xacro:insert_block name="wheel_geometry" />
-        </geometry>
-            <material name="Black">
-            <color rgba="0 0 0 1"/>
-        </material>
-   </visual>
-   <xacro:insert_block name="wheel_inertia" />
-   <collision>
-     <origin xyz="0 0 0" rpy="0 0 0"/>
-     <geometry>
-       <xacro:insert_block name="wheel_geometry" />
-     </geometry>
-   </collision>
-</link>
+<xacro:wheel name="left_rear_wheel" y_offset="${wheel_y_offset}" parent="rear_speed_link" j_type="fixed"/>
+<xacro:wheel name="right_rear_wheel" y_offset="-${wheel_y_offset}" parent="rear_speed_link" j_type="fixed"/>
 <joint name="front_steer_joint" type="revolute">
   <origin xyz="${front_wheel_x_offset} 0 ${wheel_z_offset}" rpy="0 0 0"/>
@@ -198,63 +157,13 @@
         <origin xyz="0 0 0" rpy="0 0 0" />
         <geometry>
-            <box size="0.05 0.4 0.05" />
+            <box size="0.01 0.18 0.01" />
         </geometry>
-            <material name="Cyan">
+        <material name="Cyan">
             <color rgba="0 1.0 1.0 1.0"/>
         </material>
    </visual>
 </link>
-<joint name="left_front_wheel_joint" type="continuous">
-    <origin xyz="0 ${wheel_y_offset} 0" rpy="${pi_2} 0 0"/>
-    <parent link="front_steer_link"/>
-    <child link="left_front_wheel_link"/>
-    <axis xyz="0 0 -1" />
-    <limit effort="10" velocity="100" />
-</joint>
-<xacro:wheel_transmission name="left_front_wheel" />
-<link name="left_front_wheel_link">
-    <visual>
-        <origin xyz="0 0 0" rpy="0 0 0" />
-        <geometry>
-            <xacro:insert_block name="wheel_geometry" />
-        </geometry>
-        <material name="Grey">
-            <color rgba="0.2 0.2 0.2 1"/>
-        </material>
-   </visual>
-   <xacro:insert_block name="wheel_inertia" />
-   <collision>
-     <origin xyz="0 0 0" rpy="0 0 0"/>
-     <geometry>
-       <xacro:insert_block name="wheel_geometry" />
-     </geometry>
-   </collision>
-</link>
-<xacro:wheel_transmission name="right_front_wheel" />
-<joint name="right_front_wheel_joint" type="continuous">
-    <origin xyz="0 -${wheel_y_offset} 0" rpy="${pi_2} 0 0"/>
-    <parent link="front_steer_link"/>
-    <child link="right_front_wheel_link"/>
-    <axis xyz="0 0 -1" />
-    <limit effort="10" velocity="100" />
-</joint>
-<link name="right_front_wheel_link">
-    <visual>
-        <origin xyz="0 0 0" rpy="0 0 0" />
-        <geometry>
-            <xacro:insert_block name="wheel_geometry" />
-        </geometry>
-        <material name="Grey">
-            <color rgba="0.2 0.2 0.2 1"/>
-        </material>
-   </visual>
-   <xacro:insert_block name="wheel_inertia" />
-   <collision>
-     <origin xyz="0 0 0" rpy="0 0 0"/>
-     <geometry>
-       <xacro:insert_block name="wheel_geometry" />
-     </geometry>
-   </collision>
-</link>
+<xacro:slipping_wheel name="right_front_wheel" y_offset="-${wheel_y_offset}" parent="front_steer_link" j_type="continuous"/>
+<xacro:slipping_wheel name="left_front_wheel" y_offset="${wheel_y_offset}" parent="front_steer_link" j_type="continuous"/>
 <gazebo>
   <plugin name="gazebo_ros_control" filename="libgazebo_ros_control.so">
@@ -272,8 +181,4 @@
     </plugin>
 </gazebo>
-<xacro:wheel_params link="left_rear_wheel_link"/>
-<xacro:wheel_params link="right_rear_wheel_link"/>
-<xacro:wheel_params link="left_front_wheel_link"/>
-<xacro:wheel_params link="right_front_wheel_link"/>
 <joint name="hoyuko_fixed_joint" type="fixed">
     <origin xyz="0 0 0.25" rpy="0 0 0"/>

Commit message: Debugging to match real life

File: catkin_ws/src/auto_rc_car_description/urdf/car_base.urdf.xacro (robot description, xacro)
@@ -182,5 +182,5 @@
 </gazebo>
 <joint name="hoyuko_fixed_joint" type="fixed">
-    <origin xyz="0 0 0.25" rpy="0 0 0"/>
+    <origin xyz="0 0 0.25" rpy="0 0 3.1415"/>
     <parent link="chassis_link"/>
     <child link="hoyuko_laser_link"/>

Commit message: Add visual to front of car

File: catkin_ws/src/auto_rc_car_description/urdf/car_base.urdf.xacro (robot description, xacro)
@@ -83,4 +83,13 @@
         <geometry>
             <xacro:insert_block name="chassis_geometry" />
+        </geometry>
+            <material name="Cyan">
+            <color rgba="0 1.0 1.0 1.0"/>
+        </material>
+   </visual>
+   <visual>
+        <origin xyz="0.15 0 0" rpy="0 0 0" />
+        <geometry>
+            <box size="0.08 0.08 0.08" />
         </geometry>
             <material name="Cyan">

Commit message: changes

File: catkin_ws/src/auto_rc_car_description/urdf/car_base.urdf.xacro (robot description, xacro)
@@ -191,5 +191,5 @@
 </gazebo>
 <joint name="hoyuko_fixed_joint" type="fixed">
-    <origin xyz="0 0 0.25" rpy="0 0 3.1415"/>
+    <origin xyz="0 0 0.15" rpy="0 0 3.1415"/>
     <parent link="chassis_link"/>
     <child link="hoyuko_laser_link"/>

Commit message: Uploading some test drive code

File: catkin_ws/src/auto_rc_car_description/urdf/car_base.urdf.xacro (robot description, xacro)
@@ -191,5 +191,5 @@
 </gazebo>
 <joint name="hoyuko_fixed_joint" type="fixed">
-    <origin xyz="0 0 0.15" rpy="0 0 3.1415"/>
+    <origin xyz="0 0 0.15" rpy="0 0 0"/>
     <parent link="chassis_link"/>
     <child link="hoyuko_laser_link"/>
@@ -226,18 +226,18 @@
         <scan>
           <horizontal>
-            <samples>1081</samples>
+            <samples>720</samples>
             <resolution>1</resolution>
-            <min_angle>-2.3561944902</min_angle>
-            <max_angle>2.3561944902</max_angle>
+            <min_angle>-1.57079632679</min_angle>
+            <max_angle>1.57079632679</max_angle>
           </horizontal>
         </scan>
         <range>
           <min>0.1</min>
-          <max>10.0</max>
+          <max>12.0</max>
           <resolution>0.01</resolution>
         </range>
         <noise>
           <mean>0.0</mean>
-          <stddev>0.01</stddev>
+          <stddev>0.0</stddev>
         </noise>
       </ray>

Commit message: Change to 4WD

File: catkin_ws/src/auto_rc_car_description/urdf/car_base.urdf.xacro (robot description, xacro)
@@ -21,12 +21,22 @@
    </inertial>
 </xacro:property>
-<xacro:macro name="wheel" params="name y_offset parent j_type">
+<xacro:macro name="wheel" params="name parent j_type polarity *origin">
   <joint name="${name}_joint" type="${j_type}">
-    <origin xyz="0 ${y_offset} 0" rpy="${pi_2} 0 0"/>
+    <xacro:insert_block name="origin"/>
     <parent link="${parent}"/>
     <child link="${name}_link"/>
-    <axis xyz="0 0 -1" />
+    <axis xyz="0 0 ${polarity}" />
     <limit effort="10" velocity="100" />
   </joint>
+  <transmission name="${name}_transmission" type="SimpleTransmission">
+    <type>transmission_interface/SimpleTransmission</type>
+    <joint name="${name}_joint">
+      <hardwareInterface>EffortJointInterface</hardwareInterface>
+    </joint>
+    <actuator name="${name}_joint_motor">
+      <hardwareInterface>EffortJointInterface</hardwareInterface>
+      <mechanicalReduction>1</mechanicalReduction>
+    </actuator>
+  </transmission>
   <link name="${name}_link">
     <visual>
@@ -59,17 +69,4 @@
   </gazebo>
 </xacro:macro>
-<xacro:macro name="slipping_wheel" params="name y_offset parent j_type">
-  <xacro:wheel name="${name}" y_offset="${y_offset}" parent="${parent}" j_type="${j_type}"/>
-  <transmission name="${name}_joint_transmission" type="SimpleTransmission">
-  <type>transmission_interface/SimpleTransmission</type>
-  <joint name="${name}_joint">
-    <hardwareInterface>EffortJointInterface</hardwareInterface>
-  </joint>
-  <actuator name="${name}_joint_motor">
-    <hardwareInterface>EffortJointInterface</hardwareInterface>
-    <mechanicalReduction>1</mechanicalReduction>
-  </actuator>
-</transmission>
-</xacro:macro>
 <link name="base_link"/>
 <joint name="base_joint" type="fixed">
@@ -105,39 +102,4 @@
    </collision>
 </link>
-<joint name="rear_speed_joint" type="continuous">
-  <origin xyz="${rear_wheel_x_offset} 0 ${wheel_z_offset}" rpy="0 0 0"/>
-    <parent link="chassis_link"/>
-    <child link="rear_speed_link"/>
-    <axis xyz="0 1 0" />
-    <limit effort="100" velocity="100" />
-</joint>
-<transmission name="speed_joint_transmission" type="SimpleTransmission">
-  <type>transmission_interface/SimpleTransmission</type>
-  <joint name="rear_speed_joint">
-    <hardwareInterface>EffortJointInterface</hardwareInterface>
-  </joint>
-  <actuator name="rear_speed_joint_motor">
-    <hardwareInterface>EffortJointInterface</hardwareInterface>
-    <mechanicalReduction>1</mechanicalReduction>
-  </actuator>
-</transmission>
-<link name="rear_speed_link">
-   <inertial>
-     <origin xyz="0 0 0" rpy="0 0 0"/>
-     <mass value="1"/>
-     <inertia ixx="10"  ixy="0"  ixz="0" iyy="1" iyz="0" izz="10" />
-   </inertial>
-    <visual>
-        <origin xyz="0 0 0" rpy="${pi/2.0} 0 0" />
-        <geometry>
-            <cylinder radius="0.01" length="0.18"/>
-        </geometry>
-            <material name="Cyan">
-            <color rgba="0 1.0 1.0 1.0"/>
-        </material>
-   </visual>
-</link>
-<xacro:wheel name="left_rear_wheel" y_offset="${wheel_y_offset}" parent="rear_speed_link" j_type="fixed"/>
-<xacro:wheel name="right_rear_wheel" y_offset="-${wheel_y_offset}" parent="rear_speed_link" j_type="fixed"/>
 <joint name="front_steer_joint" type="revolute">
   <origin xyz="${front_wheel_x_offset} 0 ${wheel_z_offset}" rpy="0 0 0"/>
@@ -173,6 +135,16 @@
    </visual>
 </link>
-<xacro:slipping_wheel name="right_front_wheel" y_offset="-${wheel_y_offset}" parent="front_steer_link" j_type="continuous"/>
-<xacro:slipping_wheel name="left_front_wheel" y_offset="${wheel_y_offset}" parent="front_steer_link" j_type="continuous"/>
+<xacro:wheel name="right_front_wheel" parent="front_steer_link" j_type="continuous" polarity="-1">
+  <origin xyz="0 -${wheel_y_offset} 0" rpy="${pi/2} 0 0"/>
+</xacro:wheel>
+<xacro:wheel name="left_front_wheel" parent="front_steer_link" j_type="continuous" polarity="1">
+  <origin xyz="0 ${wheel_y_offset} 0" rpy="${-pi/2} 0 0"/>
+</xacro:wheel>
+<xacro:wheel name="left_rear_wheel" parent="chassis_link" j_type="continuous" polarity="1">
+  <origin xyz="${rear_wheel_x_offset} -${wheel_y_offset} ${wheel_z_offset}" rpy="${-pi/2} 0 0"/>
+</xacro:wheel>
+<xacro:wheel name="right_rear_wheel" parent="chassis_link" j_type="continuous" polarity="-1">
+  <origin xyz="${rear_wheel_x_offset} ${wheel_y_offset} ${wheel_z_offset}" rpy="${pi/2} 0 0"/>
+</xacro:wheel>
 <gazebo>
   <plugin name="gazebo_ros_control" filename="libgazebo_ros_control.so">

Commit message: Add parameter for sensor noise

File: catkin_ws/src/auto_rc_car_description/urdf/car_base.urdf.xacro (robot description, xacro)
@@ -4,4 +4,7 @@
 mit-racecar/racecar_gazebo
 -->
+<xacro:arg name="SENSOR_NOISE" default="0.0"/>
+<xacro:include filename="$(find auto_rc_car_description/urdf/car_sensors.urdf.xacro"/>
+<xacro:macro name="car_sensors" NOISE_MAG="${SENSOR_NOISE}"/>
 <!-- Set Origin: Center of body lengthwise, height of ~middle of the gearbox -->
 <xacro:property name="wheel_y_offset" value="0.115" />
@@ -188,37 +191,4 @@
    </inertial>
 </link>
-<xacro:unless value="$(optenv DISABLE_GAZEBO_LASER false)">
-  <gazebo reference="hoyuko_laser_link">
-    <material>Gazebo/Grey</material>
-    <sensor type="ray" name="hokuyo_sensor">
-      <pose>0 0 0.0124 0 0 0</pose>
-      <visualize>false</visualize>
-      <update_rate>40</update_rate>
-      <ray>
-        <scan>
-          <horizontal>
-            <samples>1081</samples>
-            <resolution>1</resolution>
-            <min_angle>-2.3561944902</min_angle>
-            <max_angle>2.3561944902</max_angle>
-          </horizontal>
-        </scan>
-        <range>
-          <min>0.1</min>
-          <max>10.0</max>
-          <resolution>0.01</resolution>
-        </range>
-        <noise>
-          <mean>0.0</mean>
-          <stddev>0.01</stddev>
-        </noise>
-      </ray>
-      <plugin name="gazebo_ros_hokuyo_controller" filename="libgazebo_ros_laser.so">
-        <topicName>racecar/out/laser_scan</topicName>
-        <frameName>hoyuko_laser_link</frameName>
-      </plugin>
-    </sensor>
-  </gazebo>
-</xacro:unless>
   <joint name="camera_optical_joint" type="fixed">
     <!-- these values have to be these values otherwise the gazebo camera
@@ -231,45 +201,3 @@
   <link name="camera_link_optical">
   </link>
-  <gazebo reference="kinect_link">
-        <sensor name="camera" type="depth">
-        <pose>0 0 0 0 0 0</pose>
-        <visualize>true</visualize>
-        <update_rate>20</update_rate>
-        <camera>
-          <horizontal_fov>1.047198</horizontal_fov>
-          <image>
-            <width>320</width>
-            <height>240</height>
-            <format>R8G8B8</format>
-          </image>
-          <clip>
-            <near>0.05</near>
-            <far>8</far>
-          </clip>
-        </camera>
-    <plugin name="camera_plugin" filename="libgazebo_ros_openni_kinect.so">
-      <baseline>0.2</baseline>
-      <alwaysOn>true</alwaysOn>
-      <updateRate>30.0</updateRate>
-      <cameraName>sim_depth_camera</cameraName>
-      <imageTopicName>/racecar/out/stereo_camera/rgb/image</imageTopicName>
-      <cameraInfoTopicName>/racecar/out/stereo_camera/rgb/camera_info</cameraInfoTopicName>
-      <depthImageTopicName>/racecar/out/stereo_camera/depth/image</depthImageTopicName>
-      <depthImageInfoTopicName>/racecar/out/stereo_camera/depth/camera_info</depthImageInfoTopicName>
-      <pointCloudTopicName>/racecar/out/stereo_camera/depth_cloud/points</pointCloudTopicName>
-      <frameName>camera_link_optical</frameName>
-      <pointCloudCutoff>0.05</pointCloudCutoff>
-      <distortionK1>0</distortionK1>
-      <distortionK2>0</distortionK2>
-      <distortionK3>0</distortionK3>
-      <distortionT1>0</distortionT1>
-      <distortionT2>0</distortionT2>
-      <CxPrime>0</CxPrime>
-      <Cx>0</Cx>
-      <Cy>0</Cy>
-      <focalLength>0</focalLength>
-      <hackBaseline>0</hackBaseline>
-    </plugin>
-    </sensor>
-    </gazebo>
 </robot>
