Commit message: Add yaml-based params and add arg to world launch files

File: catkin_ws/src/auto_rc_car_description/urdf/car_base.urdf.xacro (robot description, xacro)
@@ -4,22 +4,29 @@
 mit-racecar/racecar_gazebo
 -->
-<xacro:arg name="SENSOR_NOISE" default="0.0"/>
-<xacro:include filename="$(find auto_rc_car_description/urdf/car_sensors.urdf.xacro"/>
-<xacro:macro name="car_sensors" NOISE_MAG="${SENSOR_NOISE}"/>
+<xacro:arg name="CONFIG_FILE" default="base_car_params.yaml"/>
+<xacro:property name="filename" value="$(find auto_rc_car_description)/config/$(arg CONFIG_FILE)"/>
+<xacro:property name="params" value="${load_yaml(filename)}"/>
+<xacro:include filename="$(find auto_rc_car_description)/urdf/car_sensors.urdf.xacro"/>
+<xacro:car_sensors PARAMS="${params}"/>
 <!-- Set Origin: Center of body lengthwise, height of ~middle of the gearbox -->
-<xacro:property name="wheel_y_offset" value="0.115" />
-<xacro:property name="wheel_z_offset" value="-0.03" />
-<xacro:property name="rear_wheel_x_offset" value="-0.14" />
-<xacro:property name="front_wheel_x_offset" value="0.14" />
+<xacro:property name="wheel_y_offset"       value="${params.get('wheel_y_offset', 0.115)}" />
+<xacro:property name="wheel_z_offset"       value="${params.get('wheel_z_offset', 0.115)}" />
+<xacro:property name="front_wheel_x_offset" value="${params.get('front_wheel_x_offset', 0.14)}" />
+<xacro:property name="rear_wheel_x_offset"  value="${params.get('rear_wheel_x_offset', -0.14)}" />
 <xacro:property name="pi_2" value="1.5708" />
 <xacro:property name="pi_4" value="0.7854" />
 <xacro:property name="chassis_geometry">
-  <box size="0.4 0.13 0.05" />
+  <box size="${params.get('chassis_length', 0.4)} ${params.get('chassis_width', 0.13)} ${params.get('chassis_height', 0.05)}" />
 </xacro:property>
 <xacro:property name="chassis_inertia">
    <inertial>
      <origin xyz="0 0 0" rpy="0 0 0"/>
-     <mass value="100"/>
-     <inertia ixx="100"  ixy="0"  ixz="0" iyy="100" iyz="0" izz="10" />
+     <mass value="${params.get('chassis_mass', 100)}"/>
+     <inertia ixx="${params.get('chassis_Ixx', 100)}"
+              ixy="${params.get('chassis_Ixy', 0)}"
+              ixz="${params.get('chassis_Ixz', 0)}"
+              iyy="${params.get('chassis_Iyy', 100)}"
+              iyz="${params.get('chassis_Iyz', 0)}"
+              izz="${params.get('chassis_Izz', 10)}" />
    </inertial>
 </xacro:property>
@@ -30,5 +37,6 @@
     <child link="${name}_link"/>
     <axis xyz="0 0 ${polarity}" />
-    <limit effort="10" velocity="100" />
+    <limit effort="${params.get('wheel_effort_limit', 10)}"
+           velocity="${params.get('wheel_velocity_limit', 10)}" />
   </joint>
   <transmission name="${name}_transmission" type="SimpleTransmission">
@@ -46,5 +54,5 @@
       <origin xyz="0 0 0" rpy="0 0 0" />
       <geometry>
-        <cylinder length="0.05" radius="0.055" />
+        <cylinder length="0.05" radius="${params.get('wheel_radius', 0.1)}" />
       </geometry>
       <material name="Black">
@@ -54,19 +62,24 @@
     <inertial>
       <origin xyz="0 0 0" rpy="0 0 0"/>
-      <mass value="1"/>
-      <inertia ixx="10"  ixy="0"  ixz="0" iyy="10" iyz="0" izz="1" />
+      <mass value="${params.get('wheel_mass', 1)}"/>
+      <inertia ixx="${params.get('wheel_Ixx', 10)}"
+               ixy="${params.get('wheel_Ixy', 0)}"
+               ixz="${params.get('wheel_Ixz', 0)}"
+               iyy="${params.get('wheel_Iyy', 1)}"
+               iyz="${params.get('wheel_Iyz', 0)}"
+               izz="${params.get('wheel_Izz', 1)}" />
     </inertial>
     <collision>
       <origin xyz="0 0 0" rpy="0 0 0"/>
       <geometry>
-        <cylinder length="0.05" radius="0.1" />
+        <cylinder length="0.05" radius="${params.get('wheel_radius', 0.1)}" />
       </geometry>
     </collision>
   </link>
     <gazebo reference="${name}_link">
-      <mu1 value="10.0"/>
-      <mu2 value="10.0"/>
-      <kp  value="10000000.0" />
-      <kd  value="5.0" />
+      <mu1 value="${params.get('wheel_gaz_mu1', 10.0)}"/>
+      <mu2 value="${params.get('wheel_gaz_mu2', 10.0)}"/>
+      <kp  value="${params.get('wheel_gaz_kp', 10000000.0)}" />
+      <kd  value="${params.get('wheel_gaz_kd', 5.0)}" />
       <material>Gazebo/Black</material>
   </gazebo>

File: catkin_ws/src/auto_rc_car_description/urdf/car_sensors.urdf.xacro (robot description, xacro)
@@ -1,5 +1,5 @@
 <?xml version="1.0"?>
 <robot name="racecar" xmlns:xacro="http://www.ros.org/wiki/xacro">
-<xacro:macro name="car_sensors" params="NOISE_MAG">
+<xacro:macro name="car_sensors" params="PARAMS">
 <xacro:unless value="$(optenv DISABLE_GAZEBO_LASER false)">
   <gazebo reference="hoyuko_laser_link">
@@ -25,5 +25,5 @@
         <noise>
           <mean>0.1</mean>
-          <stddev>${NOISE_MAG*0.5}</stddev>
+          <stddev>${PARAMS.get('lidar_noise', 0.0)}</stddev>
         </noise>
       </ray>

Commit message: Debug and set new params

File: catkin_ws/src/auto_rc_car_description/urdf/car_base.urdf.xacro (robot description, xacro)
@@ -11,7 +11,7 @@
 <!-- Set Origin: Center of body lengthwise, height of ~middle of the gearbox -->
 <xacro:property name="wheel_y_offset"       value="${params.get('wheel_y_offset', 0.115)}" />
-<xacro:property name="wheel_z_offset"       value="${params.get('wheel_z_offset', 0.115)}" />
-<xacro:property name="front_wheel_x_offset" value="${params.get('front_wheel_x_offset', 0.14)}" />
-<xacro:property name="rear_wheel_x_offset"  value="${params.get('rear_wheel_x_offset', -0.14)}" />
+<xacro:property name="wheel_z_offset"       value="${params.get('wheel_z_offset', 0.0098)}" />
+<xacro:property name="front_wheel_x_offset" value="${params.get('front_wheel_x_offset', 0.1755)}" />
+<xacro:property name="rear_wheel_x_offset"  value="${params.get('rear_wheel_x_offset', 0.1845)}" />
 <xacro:property name="pi_2" value="1.5708" />
 <xacro:property name="pi_4" value="0.7854" />
@@ -22,11 +22,11 @@
    <inertial>
      <origin xyz="0 0 0" rpy="0 0 0"/>
-     <mass value="${params.get('chassis_mass', 100)}"/>
-     <inertia ixx="${params.get('chassis_Ixx', 100)}"
+     <mass value="${params.get('chassis_mass', 3)}"/>
+     <inertia ixx="${params.get('chassis_Ixx', 3)}"
               ixy="${params.get('chassis_Ixy', 0)}"
               ixz="${params.get('chassis_Ixz', 0)}"
-              iyy="${params.get('chassis_Iyy', 100)}"
+              iyy="${params.get('chassis_Iyy', 3)}"
               iyz="${params.get('chassis_Iyz', 0)}"
-              izz="${params.get('chassis_Izz', 10)}" />
+              izz="${params.get('chassis_Izz', 3)}" />
    </inertial>
 </xacro:property>
@@ -37,6 +37,6 @@
     <child link="${name}_link"/>
     <axis xyz="0 0 ${polarity}" />
-    <limit effort="${params.get('wheel_effort_limit', 10)}"
-           velocity="${params.get('wheel_velocity_limit', 10)}" />
+    <limit effort="${params.get('motor_effort_limit', 0.9730)*params.get('drivetrain_radius_b', 0.0413) / params.get('drivetrain_radius_a', 0.01605)}"
+           velocity="${params.get('car_velocity_limit', 15) / params.get('wheel_radius', 0.06)}" />
   </joint>
   <transmission name="${name}_transmission" type="SimpleTransmission">
@@ -54,5 +54,5 @@
       <origin xyz="0 0 0" rpy="0 0 0" />
       <geometry>
-        <cylinder length="0.05" radius="${params.get('wheel_radius', 0.1)}" />
+        <cylinder length="0.05" radius="${params.get('wheel_radius', 0.06)}" />
       </geometry>
       <material name="Black">
@@ -62,16 +62,16 @@
     <inertial>
       <origin xyz="0 0 0" rpy="0 0 0"/>
-      <mass value="${params.get('wheel_mass', 1)}"/>
-      <inertia ixx="${params.get('wheel_Ixx', 10)}"
+      <mass value="${params.get('wheel_mass', 0.01)}"/>
+      <inertia ixx="${params.get('wheel_Ixx', 0.0008)}"
                ixy="${params.get('wheel_Ixy', 0)}"
                ixz="${params.get('wheel_Ixz', 0)}"
-               iyy="${params.get('wheel_Iyy', 1)}"
+               iyy="${params.get('wheel_Iyy', 0.00001)}"
                iyz="${params.get('wheel_Iyz', 0)}"
-               izz="${params.get('wheel_Izz', 1)}" />
+               izz="${params.get('wheel_Izz', 0.00001)}" />
     </inertial>
     <collision>
       <origin xyz="0 0 0" rpy="0 0 0"/>
       <geometry>
-        <cylinder length="0.05" radius="${params.get('wheel_radius', 0.1)}" />
+        <cylinder length="0.05" radius="${params.get('wheel_radius', 0.06)}" />
       </geometry>
     </collision>

Commit message: Test and try to fix params

File: catkin_ws/src/auto_rc_car_description/urdf/car_base.urdf.xacro (robot description, xacro)
@@ -119,5 +119,5 @@
 </link>
 <joint name="front_steer_joint" type="revolute">
-  <origin xyz="${front_wheel_x_offset} 0 ${wheel_z_offset}" rpy="0 0 0"/>
+  <origin xyz="${-front_wheel_x_offset} 0 ${wheel_z_offset}" rpy="0 0 0"/>
     <parent link="chassis_link"/>
     <child link="front_steer_link"/>
@@ -158,8 +158,8 @@
 </xacro:wheel>
 <xacro:wheel name="left_rear_wheel" parent="chassis_link" j_type="continuous" polarity="1">
-  <origin xyz="${rear_wheel_x_offset} -${wheel_y_offset} ${wheel_z_offset}" rpy="${-pi/2} 0 0"/>
+  <origin xyz="${-rear_wheel_x_offset} -${wheel_y_offset} ${wheel_z_offset}" rpy="${-pi/2} 0 0"/>
 </xacro:wheel>
 <xacro:wheel name="right_rear_wheel" parent="chassis_link" j_type="continuous" polarity="-1">
-  <origin xyz="${rear_wheel_x_offset} ${wheel_y_offset} ${wheel_z_offset}" rpy="${pi/2} 0 0"/>
+  <origin xyz="${-rear_wheel_x_offset} ${wheel_y_offset} ${wheel_z_offset}" rpy="${pi/2} 0 0"/>
 </xacro:wheel>
 <gazebo>

Commit message: Commit current state, not working yet

File: catkin_ws/src/auto_rc_car_description/urdf/car_base.urdf.xacro (robot description, xacro)
@@ -101,5 +101,5 @@
         </material>
    </visual>
-   <visual>
+   <!-- <visual>
         <origin xyz="0.15 0 0" rpy="0 0 0" />
         <geometry>
@@ -109,5 +109,5 @@
             <color rgba="0 1.0 1.0 1.0"/>
         </material>
-   </visual>
+   </visual> -->
     <xacro:insert_block name="chassis_inertia" />
    <collision>
@@ -123,5 +123,5 @@
     <child link="front_steer_link"/>
     <axis xyz="0 0 1" />
-    <limit upper="0.5" lower="-0.5" effort="100" velocity="10" />
+    <limit upper="0.5" lower="-0.5" effort="2" velocity="2" />
 </joint>
 <transmission name="steer_joint_transmission" type="SimpleTransmission">
@@ -138,6 +138,6 @@
    <inertial>
      <origin xyz="0 0 0" rpy="0 0 0"/>
-     <mass value="1"/>
-     <inertia ixx="10"  ixy="0"  ixz="0" iyy="10" iyz="0" izz="1" />
+     <mass value="0.04"/>
+     <inertia ixx="0.00001"  ixy="0"  ixz="0" iyy="0.00001" iyz="0" izz="0.00001" />
    </inertial>
     <visual>
@@ -178,39 +178,3 @@
     </plugin>
 </gazebo>
-<joint name="hoyuko_fixed_joint" type="fixed">
-    <origin xyz="0 0 0.15" rpy="0 0 3.1415"/>
-    <parent link="chassis_link"/>
-    <child link="hoyuko_laser_link"/>
-    <axis xyz="0 0 1" />
-</joint>
-<link name="hoyuko_laser_link">
-   <inertial>
-     <origin xyz="0 0 0" rpy="0 0 0"/>
-     <mass value="1"/>
-     <inertia ixx="10"  ixy="0"  ixz="0" iyy="10" iyz="0" izz="1" />
-   </inertial>
-</link>
-<joint name="kinect_fixed_joint" type="fixed">
-    <origin xyz="0 0 0.25" rpy="0 0 0"/>
-    <parent link="chassis_link"/>
-    <child link="kinect_link"/>
-    <axis xyz="0 0 1" />
-</joint>
-<link name="kinect_link">
-   <inertial>
-     <origin xyz="0 0 0" rpy="0 0 0"/>
-     <mass value="1"/>
-     <inertia ixx="10"  ixy="0"  ixz="0" iyy="10" iyz="0" izz="1" />
-   </inertial>
-</link>
-  <joint name="camera_optical_joint" type="fixed">
-    <!-- these values have to be these values otherwise the gazebo camera
-        image won't be aligned properly with the frame it is supposedly
-        originating from -->
-    <origin xyz="0 0 0" rpy="${-pi/2} 0 ${-pi/2}"/>
-    <parent link="kinect_link"/>
-    <child link="camera_link_optical"/>
-  </joint>
-  <link name="camera_link_optical">
-  </link>
 </robot>
